Commit message: paolo

File: urdf/ur5_lab_standalone.urdf.xacro (robot description, xacro)
@@ -8,5 +8,5 @@
   <xacro:include filename="$(find robotiq_ft_sensor)/urdf/robotiq_ft300.urdf.xacro" />
   <xacro:robotiq_ft300 parent="ur5_wrist_3_link" prefix="">
-      <origin xyz="0 0 0" rpy="0 0 0"/>
+      <origin xyz="0 0 0" rpy="0 0 -1.5707"/>
   </xacro:robotiq_ft300>
  <!-- <joint name="wl3_tip" type="fixed">

Commit message: paolo: impedeze funzionanti

File: urdf/ur5_lab_standalone.urdf.xacro (robot description, xacro)
@@ -8,5 +8,5 @@
   <xacro:include filename="$(find robotiq_ft_sensor)/urdf/robotiq_ft300.urdf.xacro" />
   <xacro:robotiq_ft300 parent="ur5_wrist_3_link" prefix="">
-      <origin xyz="0 0 0" rpy="0 0 -1.5707"/>
+      <origin xyz="0 0 0" rpy="0 0 3.1415"/>
   </xacro:robotiq_ft300>
  <!-- <joint name="wl3_tip" type="fixed">

Commit message: paolo: topic simple touch

File: urdf/ur5_lab_standalone.urdf.xacro (robot description, xacro)
@@ -8,5 +8,5 @@
   <xacro:include filename="$(find robotiq_ft_sensor)/urdf/robotiq_ft300.urdf.xacro" />
   <xacro:robotiq_ft300 parent="ur5_wrist_3_link" prefix="">
-      <origin xyz="0 0 0" rpy="0 0 3.1415"/>
+      <origin xyz="0 0 0" rpy="0 0 0"/>
   </xacro:robotiq_ft300>
  <!-- <joint name="wl3_tip" type="fixed">
